File: 48tsop-32dip.kicad_pcb (KiCad board)
At the start: 2 copper layers, 41.1 x 15.2 mm, 5 parts, among them U1 AM29F400Bx-xxEx, U2 27C040/020/010

Commit message: gerbers
Other:
- board text added: "A18"
- board text added: "~{CE}"
- board text added: "~{OE}"
Changed lines of the file:
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@@
-		)
-		(fp_line
-			(start -1.4 -1)
-			(end 1.4 -1)
-			(stroke
-				(width 0.12)
-				(type solid)
-			)
-			(layer "F.SilkS")
-		)
-		(fp_line
-			(start -1.4 1)
-			(end -1.4 -1)
-			(stroke
-				(width 0.12)
-				(type solid)
-			)
-			(layer "F.SilkS")
-		)
-		(fp_line
-			(start 1.4 -1)
-			(end 1.4 1)
-			(stroke
-				(width 0.12)
-				(type solid)
-			)
-			(layer "F.SilkS")
-		)
-		(fp_line
-			(start 1.4 1)
-			(end -1.4 1)
-			(stroke
-				(width 0.12)
-				(type solid)
-			)
-			(layer "F.SilkS")
 		)
 		(fp_line
@@
 		)
 		(fp_line
-			(start 1.4 1)
-			(end -1.4 1)
-			(stroke
-				(width 0.12)
-				(type solid)
-			)
-			(layer "F.SilkS")
-		)
-		(fp_line
-			(start 1.4 -1)
-			(end 1.4 1)
-			(stroke
-				(width 0.12)
-				(type solid)
-			)
-			(layer "F.SilkS")
-		)
-		(fp_line
-			(start -1.4 1)
-			(end -1.4 -1)
-			(stroke
-				(width 0.12)
-				(type solid)
-			)
-			(layer "F.SilkS")
-		)
-		(fp_line
-			(start -1.4 -1)
-			(end 1.4 -1)
-			(stroke
-				(width 0.12)
-				(type solid)
-			)
-			(layer "F.SilkS")
-		)
-		(fp_line
 			(start 1.65 1.25)
 			(end 1.65 -1.25)
@@
 		(property "Reference" "JP3"
 			(at 0 -1.8 0)
-			(layer "F.SilkS")
+			(layer "F.Fab")
 			(effects
 				(font
@@
 		)
 		(fp_line
-			(start -1.4 -1)
-			(end 1.4 -1)
-			(stroke
-				(width 0.12)
-				(type solid)
-			)
-			(layer "F.SilkS")
-		)
-		(fp_line
-			(start -1.4 1)
-			(end -1.4 -1)
-			(stroke
-				(width 0.12)
-				(type solid)
-			)
-			(layer "F.SilkS")
-		)
-		(fp_line
-			(start 1.4 -1)
-			(end 1.4 1)
-			(stroke
-				(width 0.12)
-				(type solid)
-			)
-			(layer "F.SilkS")
-		)
-		(fp_line
-			(start 1.4 1)
-			(end -1.4 1)
-			(stroke
-				(width 0.12)
-				(type solid)
-			)
-			(layer "F.SilkS")
-		)
-		(fp_line
 			(start -1.65 -1.25)
 			(end -1.65 1.25)
@@
 		(fill no)
 		(layer "F.Fab")
+	)
+	(gr_text "~{CE}"
+		(at 109.728 91.313 0)
+		(layer "F.SilkS")
+		(effects
+			(font
+				(size 0.7 0.7)
+				(thickness 0.14)
+				(bold yes)
+			)
+			(justify left)
+		)
 	)
 	(gr_text "4Mbit 29F400\n2Mbit 29F200\n1Mbit 29F100"
@@
 		)
 	)
+	(gr_text "A18"
+		(at 79.629 91.567 0)
+		(layer "F.SilkS")
+		(effects
+			(font
+				(size 0.7 0.7)
+				(thickness 0.14)
+				(bold yes)
+			)
+			(justify left)
+		)
+	)
 	(gr_text "Pin 1 Bottom of Chip"
 		(at 75.25 80.5 0)
@@
 		)
 	)
+	(gr_text "~{OE}"
+		(at 109.601 81.407 0)
+		(layer "F.SilkS")
+		(effects
+			(font
+				(size 0.7 0.7)
+				(thickness 0.14)
+				(bold yes)
+			)
+			(justify left)
+		)
+	)

Commit message: a
Other:
- board text added: "github.com/owen-rp2a03/smd_eeprom_adapter"
Changed lines of the file:
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@@
+		)
+	)
+	(gr_text "github.com/owen-rp2a03/smd_eeprom_adapter"
+		(at 115.189 86.36 90)
+		(layer "F.SilkS")
+		(effects
+			(font
+				(size 0.5 0.375)
+				(thickness 0.075)
+				(bold yes)
+			)
+			(justify bottom)
 		)
 	)

Commit message: fix gerber
Other:
- board text added: "github.com/owen-rp2a03/ smd_eeprom_adapter"
- board text removed: "github.com/owen-rp2a03/smd_eeprom_adapter"
Changed lines of the file:
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@@
 		)
 	)
-	(gr_text "github.com/owen-rp2a03/smd_eeprom_adapter"
-		(at 115.189 86.36 90)
+	(gr_text "github.com/owen-rp2a03/\n			smd_eeprom_adapter"
+		(at 115.443 87.249 90)
 		(layer "F.SilkS")
 		(effects
 			(font
-				(size 0.5 0.375)
-				(thickness 0.075)
+				(size 0.6 0.55)
+				(thickness 0.1)
 				(bold yes)
 			)
